File: Atmega1284P_New.brd (EAGLE design)
At the start: 69.5 x 53.3 mm, 49 parts, among them U2 ATMEGA1284P-AU, U3 ESP-WROOM-32

Commit message: GOOD_Working_Copy
Parts:
- removed C10, C7, C8, C9: 0.1uf, SparkFun-Passives:0805
- removed C4, C5: (no value), SparkFun-Passives:0805
- removed I2C, SERIAL1: (no value), SparkFun-Connectors:1X06
- removed JTAG: (no value), SparkFun-Connectors:AVR_ICSP
- removed LED-CON, RESET: (no value), SparkFun-Connectors:1X02@1
- removed LED2: (no value), adafruit:CHIPLED_0805
- removed P-ACD, PB0-7: (no value), SparkFun-Connectors:2X5
- removed PA0-3: (no value), SparkFun-Connectors:1X04
- removed R-LED: 220, resistor:R0805
- removed R4, R6, R7: 10k, resistor:R0805
- removed U2: ATMEGA1284P-AU, Atmel_By_element14_Batch_1-00:QFP80P1200X1200X120-44N
- removed Y2: (no value), SparkFun-Clocks:CRYSTAL-SMD-5X3.2-2PAD
- moved R-IOW 50.0 mm to (58.4, 16.5)
- moved 3.3V 30.5 mm to (33.0, 45.7)
- moved SERIALW 27.4 mm to (21.6, 38.1)
- moved IO0 26.9 mm to (43.2, 45.7)
- moved C11 26.7 mm to (76.2, 21.6)
- moved I2CW 26.2 mm to (27.9, 35.6)
- moved LED_IOW 25.4 mm to (77.5, 29.2)
- moved U3 22.9 mm to (41.9, 30.5)
- moved C6 21.6 mm to (55.9, 24.1)
- moved C12 20.9 mm to (59.7, 33.0)
- moved PWR1 20.1 mm to (64.8, 61.0)
- moved PWR2 19.4 mm to (64.8, 54.6)
- moved R5 18.0 mm to (61.0, 25.4)
- moved SERIAL0 16.1 mm to (68.6, 26.7)
- moved SER0_RX 6.35 mm to (57.1, 40.6)
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Connections:
- removed net N$10: JTAG.1, U2.21
- removed net N$11: JTAG.5, U2.22
- removed net N$12: JTAG.9, U2.24
- removed net N$14: C4.2, U2.8, Y2.P$1
- removed net N$15: PA0-3.4, U2.37
- removed net N$16: PA0-3.3, U2.36
- removed net N$17: PA0-3.2, U2.35
- removed net N$18: PA0-3.1, U2.34
- removed net N$19: LED-CON.1, R-LED.1
- removed net N$2: PB0-7.3, U2.43
- removed net N$20: LED2.A, R-LED.2
- removed net N$21: I2C.1, I2C.3, R6.1, U2.19
- removed net N$22: I2C.2, I2C.4, R7.1, U2.20
- removed net N$23: PB0-7.1, U2.40
- removed net N$24: PB0-7.2, U2.41
- removed net N$25: PB0-7.4, U2.42
- removed net N$26: PB0-7.8, U2.3
- removed net N$27: PB0-7.5, U2.1
- removed net N$28: PB0-7.6, U2.44
- removed net N$29: PB0-7.7, U2.2
- removed net N$30: JTAG.6, R4.1, RESET.2, U2.4
- removed net N$31: P-ACD.9, U2.26
- removed net N$32: P-ACD.7, U2.25
- removed net N$33: P-ACD.5, U2.16
- removed net N$34: P-ACD.3, U2.15
- removed net N$35: P-ACD.1, U2.14
- removed net N$36: P-ACD.2, U2.13
- removed net N$37: P-ACD.10, U2.30
- removed net N$38: P-ACD.8, U2.31
- removed net N$39: P-ACD.6, U2.32
- removed net N$4: C10.1, U2.29
- removed net N$40: LED-CON.2, P-ACD.4, U2.33
- removed net N$6: C5.2, U2.7, Y2.P$2
- removed net N$7: SERIAL1.4, U2.11
- removed net N$8: SERIAL1.5, U2.12
- removed net N$9: JTAG.3, U2.23
- net GND: no longer C10.2, C4.1, C5.1, C7.2, C8.2, C9.2, I2C.5, JTAG.10, JTAG.2, LED2.C, PB0-7.10, RESET.1, SERIAL1.1, U2.18, U2.28, U2.39, U2.6
- net N$3: no longer U2.9
- net N$5: no longer U2.10
- net VCC: no longer C7.1, C8.1, C9.1, I2C.6, JTAG.4, PB0-7.9, R4.2, R6.2, R7.2, U2.17, U2.27, U2.38, U2.5
Routing:
- net GND: track 351.2 -> 0.00 mm, vias 9 -> 0
- net VCC: track 248.4 -> 0.00 mm, vias 7 -> 0
- net N$34: track 115.4 -> 0.00 mm, vias 2 -> 0
- net N$18: track 80.0 -> 0.00 mm, vias 5 -> 0
- net N$5: track 80.0 -> 0.00 mm, vias 4 -> 0
- net N$46: track 79.8 -> 0.00 mm, vias 2 -> 0
- net N$36: track 73.7 -> 0.00 mm, vias 3 -> 0
- net N$31: track 72.7 -> 0.00 mm, vias 2 -> 0
- net N$15: track 69.3 -> 0.00 mm, vias 4 -> 0
- net N$35: track 68.9 -> 0.00 mm, vias 7 -> 0
- net N$3: track 61.5 -> 0.00 mm, vias 3 -> 0
- net N$32: track 60.6 -> 0.00 mm, vias 4 -> 0
- net N$33: track 53.5 -> 0.00 mm, vias 3 -> 0
- net N$42: track 51.3 -> 0.00 mm
- net N$25: track 50.4 -> 0.00 mm, vias 4 -> 0
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
Commit message: Working Copy
Parts:
- moved SERIALW 87.5 mm to (99.1, 78.7), turned to 0 degrees
- moved 3.3V 62.7 mm to (92.7, 26.7)
- moved I2CW 59.7 mm to (87.6, 38.1), turned to 0 degrees
- moved R-IOW 59.2 mm to (106.7, 50.8)
- moved IO0 56.4 mm to (95.2, 67.3)
- moved U3 50.4 mm to (80.0, 63.5), turned to 90 degrees
- moved C11 47.7 mm to (44.5, 57.1), turned to 0 degrees
- moved R1 39.5 mm to (76.2, 34.3)
- moved R1-PWR 37.5 mm to (63.5, 71.1)
- moved C6 33.4 mm to (50.8, 57.1), turned to 0 degrees
- moved C12 32.7 mm to (52.1, 64.8), turned to 0 degrees
- moved R2 31.5 mm to (68.6, 34.3)
- moved PWR2 30.5 mm to (35.6, 45.7)
- moved PWR1 29.2 mm to (35.6, 62.2)
- moved LED_IOW 25.7 mm to (102.9, 25.4), turned to 0 degrees
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Other:
- board size 69.5 x 53.3 mm -> 160 x 100 mm
